Commit message: add rp lidar meshes, fixed casters names

File: urdf/osumy.urdf.xacro (robot description, xacro)
@@ -43,10 +43,10 @@
             <parent link="base_link"/>
             <child link="left_wheel"/>
-            <origin xyz="0.065 0.16515 -0.017" rpy="1.570796327 0 0"/>
+            <origin xyz="0.065 0.16515 -0.017" rpy="${M_PI/2} 0 0"/>
     </joint>
     <link name="left_wheel">
         <origin xyz="0 -0.0215785030951042 0" rpy="0 0 0" />
         <visual>
-                <origin xyz="0.0 0.0 0.0" rpy="-1.570796327 0 0"/>
+                <origin xyz="0.0 0.0 0.0" rpy="-${M_PI/2} 0 0"/>
                 <geometry>
                     <mesh filename="package://osumy_description/meshes/LW_Link.STL"/>
@@ -67,10 +67,10 @@
             <parent link="base_link"/>
             <child link="right_wheel"/>
-            <origin xyz="0.065 -0.16515 -0.017" rpy="1.570796327 0 0"/>
+            <origin xyz="0.065 -0.16515 -0.017" rpy="${M_PI/2} 0 0"/>
     </joint>
     <link name="right_wheel">
         <origin xyz="0 0.0215785030951041 -5.55111512312578E-17" rpy="0 0 0" />
         <visual>
-                <origin xyz="0.0 0.0 0.0" rpy="-1.570796327 0 0"/>
+                <origin xyz="0.0 0.0 0.0" rpy="-${M_PI/2} 0 0"/>
                 <geometry>
                     <mesh filename="package://osumy_description/meshes/RW_Link.STL"/>
@@ -84,4 +84,51 @@
                 <geometry>
                     <mesh filename="package://osumy_description/meshes/RW_Link.STL"/>
+                </geometry>
+            </collision>
+    </link>
+    <!-- Back Caster Wheel -->
+    <joint name="base_link_bs_joint" type="fixed">
+            <parent link="base_link"/>
+            <child link="bs_link"/>
+            <origin xyz="-0.185 0 -0.002" rpy="0 0 0"/>
+    </joint>
+    <link name="bs_link">
+        <origin xyz="-0.0143500705022477 0.00692729007829129 -0.0369933174670841" rpy="0 0 0" />
+        <visual>
+                <origin xyz="0.0 0.0 0.0" rpy="0 0 0"/>
+                <geometry>
+                    <mesh filename="package://osumy_description/meshes/BS_Link.STL"/>
+                </geometry>
+                <material name="">
+                    <color rgba="0.792156862745098 0.819607843137255 0.933333333333333 1" />
+                </material>
+            </visual>
+            <collision>
+                <origin xyz="0 0 0" rpy="0 0 0"/>
+                <geometry>
+                    <mesh filename="package://osumy_description/meshes/BS_Link.STL"/>
+                </geometry>
+            </collision>
+    </link>
+    <joint name="bs_back_caster_joint" type="fixed">
+            <parent link="bs_link"/>
+            <child link="back_caster"/>
+            <origin xyz="-0.0351188870758264 0.0169606536004725 -0.0700341016151377" rpy="0 0 0"/>
+    </joint>
+    <link name="back_caster">
+        <origin xyz="-5.55111512312578E-17 0 -2.77555756156289E-17" rpy="0 0 0" />
+        <visual>
+                <origin xyz="0.0 0.0 0.0" rpy="0 0 0"/>
+                <geometry>
+                    <mesh filename="package://osumy_description/meshes/BW_Link.STL"/>
+                </geometry>
+                <material name="">
+                    <color rgba="0.792156862745098 0.819607843137255 0.933333333333333 1" />
+                </material>
+            </visual>
+            <collision>
+                <origin xyz="0 0 0" rpy="0 0 0"/>
+                <geometry>
+                    <mesh filename="package://osumy_description/meshes/BW_Link.STL"/>
                 </geometry>
             </collision>
@@ -91,21 +138,21 @@
             <parent link="base_link"/>
             <child link="fs_link"/>
-            <origin xyz="-0.185 0 -0.002" rpy="0 0 0"/>
+            <origin xyz="0.185 0 -0.002" rpy="0 0 0"/>
     </joint>
     <link name="fs_link">
-        <origin xyz="-0.0143500705022477 0.00692729007829129 -0.0369933174670841" rpy="0 0 0" />
-        <visual>
-                <origin xyz="0.0 0.0 0.0" rpy="0 0 0"/>
-                <geometry>
-                    <mesh filename="package://osumy_description/meshes/BS_Link.STL"/>
-                </geometry>
-                <material name="">
-                    <color rgba="0.792156862745098 0.819607843137255 0.933333333333333 1" />
-                </material>
-            </visual>
-            <collision>
-                <origin xyz="0 0 0" rpy="0 0 0"/>
-                <geometry>
-                    <mesh filename="package://osumy_description/meshes/BS_Link.STL"/>
+        <origin xyz="-0.00871161814073018 0.0133420401993786 -0.0369931849655494" rpy="0 0 0" />
+        <visual>
+                <origin xyz="0.0 0.0 0.0" rpy="0 0 0"/>
+                <geometry>
+                    <mesh filename="package://osumy_description/meshes/FS_Link.STL"/>
+                </geometry>
+                <material name="">
+                    <color rgba="0.792156862745098 0.819607843137255 0.933333333333333 1" />
+                </material>
+            </visual>
+            <collision>
+                <origin xyz="0 0 0" rpy="0 0 0"/>
+                <geometry>
+                    <mesh filename="package://osumy_description/meshes/FS_Link.STL"/>
                 </geometry>
             </collision>
@@ -114,54 +161,7 @@
             <parent link="fs_link"/>
             <child link="front_caster"/>
-            <origin xyz="-0.0351188870758264 0.0169606536004725 -0.0700341016151377" rpy="0 0 0"/>
+            <origin xyz="-0.0213164011571543 0.0326590116462066 -0.0700341016151377" rpy="0 0 0"/>
     </joint>
     <link name="front_caster">
-        <origin xyz="-5.55111512312578E-17 0 -2.77555756156289E-17" rpy="0 0 0" />
-        <visual>
-                <origin xyz="0.0 0.0 0.0" rpy="0 0 0"/>
-                <geometry>
-                    <mesh filename="package://osumy_description/meshes/BW_Link.STL"/>
-                </geometry>
-                <material name="">
-                    <color rgba="0.792156862745098 0.819607843137255 0.933333333333333 1" />
-                </material>
-            </visual>
-            <collision>
-                <origin xyz="0 0 0" rpy="0 0 0"/>
-                <geometry>
-                    <mesh filename="package://osumy_description/meshes/BW_Link.STL"/>
-                </geometry>
-            </collision>
-    </link>
-    <!-- Back Caster Wheel -->
-    <joint name="base_link_bs_joint" type="fixed">
-            <parent link="base_link"/>
-            <child link="bs_link"/>
-            <origin xyz="0.185 0 -0.002" rpy="0 0 0"/>
-    </joint>
-    <link name="bs_link">
-        <origin xyz="-0.00871161814073018 0.0133420401993786 -0.0369931849655494" rpy="0 0 0" />
-        <visual>
-                <origin xyz="0.0 0.0 0.0" rpy="0 0 0"/>
-                <geometry>
-                    <mesh filename="package://osumy_description/meshes/FS_Link.STL"/>
-                </geometry>
-                <material name="">
-                    <color rgba="0.792156862745098 0.819607843137255 0.933333333333333 1" />
-                </material>
-            </visual>
-            <collision>
-                <origin xyz="0 0 0" rpy="0 0 0"/>
-                <geometry>
-                    <mesh filename="package://osumy_description/meshes/FS_Link.STL"/>
-                </geometry>
-            </collision>
-    </link>
-    <joint name="bs_front_caster_joint" type="fixed">
-            <parent link="bs_link"/>
-            <child link="back_caster"/>
-            <origin xyz="-0.0213164011571543 0.0326590116462066 -0.0700341016151377" rpy="0 0 0"/>
-    </joint>
-    <link name="back_caster">
         <origin xyz="1.11022302462516E-16 1.11022302462516E-16 8.32667268468867E-17" rpy="0 0 0" />
         <visual>
@@ -194,57 +194,34 @@
             <parent link="base_link"/>
             <child link="front_lidar"/>
-            <origin xyz="0.26135 0.00018242 0.16358" rpy="0 0 1.570796327"/>
+            <origin xyz="0.25831 -0.00051464 0.18108" rpy="0 0 ${M_PI/2}"/>
     </joint>
     <link name="front_lidar">
-        <origin xyz="-0.00845402605471413 0.000303456837048188 -0.00143540968894312" rpy="0 0 0" />
-        <visual>
-                <origin xyz="0.0 0.0 0.0" rpy="0 0 -1.570796327"/>
-                <geometry>
-                    <mesh filename="package://osumy_description/meshes/FL_LInk.STL"/>
-                </geometry>
-                <material name="">
-                    <color rgba="0.792156862745098 0.819607843137255 0.933333333333333 1" />
-                </material>
-            </visual>
-            <collision>
-                <origin xyz="0 0 0" rpy="0 0 0"/>
-                <geometry>
-                    <mesh filename="package://osumy_description/meshes/FL_LInk.STL"/>
-                </geometry>
-            </collision>
-    </link>
-    <!-- <joint name="rp_front_lidar_joint" type="fixed">
-            <parent link="front_lidar"/>
-            <child link="frp"/>
-            <origin xyz="0.0 0.0 0.0" rpy="0 0 0"/>
-    </joint>
-    <link name="frp">
-        <origin xyz="0.0 0.0 0.0" rpy="0 0 0" />
-        <visual>
-                <origin xyz="0.0 0.0 0.0" rpy="0 0 -3.1415926535897931"/>
-                <geometry>
-                    <mesh filename="package://osumy_description/meshes/rp_lidar.stl" scale="0.001 0.001 0.001"/>
-                </geometry>
-                <material name="">
-                    <color rgba="0.792156862745098 0.819607843137255 0.933333333333333 1" />
-                </material>
-            </visual>
-            <collision>
-                <origin xyz="0 0 0" rpy="0 0 0"/>
-                <geometry>
-                    <mesh filename="package://osumy_description/meshes/rp_lidar.stl" scale="0.001 0.001 0.001"/>
-                </geometry>
-            </collision>
-    </link> -->
+        <origin xyz="-0.0121634647425742 0.000482027459920101 -0.0287648483006457" rpy="0 0 0" />
+        <visual>
+                <origin xyz="0.0 0.0 0.0" rpy="0 0 ${M_PI}"/>
+                <geometry>
+                    <mesh filename="package://osumy_description/meshes/FL_Link.STL"/>
+                </geometry>
+                <material name="">
+                    <color rgba="0.792156862745098 0.819607843137255 0.933333333333333 1" />
+                </material>
+            </visual>
+            <collision>
+                <origin xyz="0 0 0" rpy="0 0 0"/>
+                <geometry>
+                    <mesh filename="package://osumy_description/meshes/FL_Link.STL"/>
+                </geometry>
+            </collision>
+    </link>
     <!-- Back Rplidar A1 -->
     <joint name="base_link_back_lidar_joint" type="fixed">
             <parent link="base_link"/>
             <child link="back_lidar"/>
-            <origin xyz="-0.26135 0.00018243 0.16358" rpy="0 0 1.570796327"/>
+            <origin xyz="-0.28054 -0.00061459 0.18108" rpy="0 0 ${M_PI/2}"/>
     </joint>
     <link name="back_lidar">
-        <origin xyz="0.0084540260547141 -0.000668307086464481 -0.00143581657171132" rpy="0 0 0" />
-        <visual>
-                <origin xyz="0.0 0.0 0.0" rpy="0 0 -1.570796327"/>
+        <origin xyz="0.0121634643954264 -0.000482027074843318 -0.028764848371282" rpy="0 0 0" />
+        <visual>
+                <origin xyz="0.0 0.0 0.0" rpy="0 0 0"/>
                 <geometry>
                     <mesh filename="package://osumy_description/meshes/BL_Link.STL"/>
@@ -261,32 +238,9 @@
             </collision>
     </link>
-    <!-- <joint name="rp_back_lidar_joint" type="fixed">
-            <parent link="back_lidar"/>
-            <child link="brp"/>
-            <origin xyz="0.0 0.0 0.0" rpy="0 0 0"/>
-    </joint>
-    <link name="brp">
-        <origin xyz="0.0 0.0 0.0" rpy="0 0 0" />
-        <visual>
-                <origin xyz="0.0 0.0 0.0" rpy="0 0 -3.1415926535897931"/>
-                <geometry>
-                    <mesh filename="package://osumy_description/meshes/rp_lidar.stl" scale="0.001 0.001 0.001"/>
-                </geometry>
-                <material name="">
-                    <color rgba="0.792156862745098 0.819607843137255 0.933333333333333 1" />
-                </material>
-            </visual>
-            <collision>
-                <origin xyz="0 0 0" rpy="0 0 0"/>
-                <geometry>
-                    <mesh filename="package://osumy_description/meshes/rp_lidar.stl" scale="0.001 0.001 0.001"/>
-                </geometry>
-            </collision>
-    </link> -->
     <!-- Realsense D435i  -->
     <joint name="base_link_back_rs_camera_joint" type="fixed">
             <parent link="base_link"/>
             <child link="rs_camera"/>
-            <origin xyz="-0.316902261320869 0 0.10208012727996" rpy="0 0 3.1415926535897931"/>
+            <origin xyz="-0.316902261320869 0 0.10208012727996" rpy="0 0 ${M_PI}"/>
     </joint>
     <link name="rs_camera">
